Commit message: Updated emotion sound and random personality

File: urdf/pidog.urdf.xacro (robot description, xacro)
@@ -1,80 +1,98 @@
 <?xml version="1.0"?>
-<robot name="pidog" xmlns:xacro="http://www.ros.org/wiki/xacro">
+<robot name="pidog" xmlns:xacro="http://www.ros.org/wiki/xacro" xmlns:gazebo="http://gazebosim.org/schemas/gazebo">
   <!-- ==================== Constants ==================== -->
-  <!-- Body dimensions based on actual PiDog -->
-  <xacro:property name="body_length" value="0.22" />
-  <xacro:property name="body_width" value="0.13" />
-  <xacro:property name="body_height" value="0.055" />
-  <xacro:property name="body_mass" value="0.9" />
-  <!-- Leg segment dimensions (adjusted for realistic stance) -->
-  <xacro:property name="upper_leg_length" value="0.085" />
-  <xacro:property name="lower_leg_length" value="0.095" />
-  <xacro:property name="leg_width" value="0.03" />
-  <xacro:property name="leg_mass" value="0.05" />
-  <!-- Head dimensions (more dog-like) -->
-  <xacro:property name="head_length" value="0.09" />
-  <xacro:property name="head_width" value="0.075" />
-  <xacro:property name="head_height" value="0.065" />
-  <xacro:property name="snout_length" value="0.04" />
-  <xacro:property name="head_mass" value="0.18" />
-  <!-- Hip joint offsets (positioned for realistic stance) -->
-  <xacro:property name="hip_front_offset_x" value="0.085" />
-  <xacro:property name="hip_hind_offset_x" value="-0.085" />
-  <xacro:property name="hip_offset_y" value="0.065" />
+  <!-- Body dimensions (based on actual PiDog) -->
+  <xacro:property name="body_length" value="0.18" />
+  <xacro:property name="body_width" value="0.10" />
+  <xacro:property name="body_height" value="0.045" />
+  <xacro:property name="body_mass" value="0.75" />
+  <!-- Leg dimensions -->
+  <xacro:property name="upper_leg_length" value="0.075" />
+  <xacro:property name="lower_leg_length" value="0.085" />
+  <xacro:property name="leg_width" value="0.028" />
+  <xacro:property name="leg_mass" value="0.06" />
+  <!-- Joint positions (shoulder/hip on body sides) -->
+  <xacro:property name="hip_front_offset_x" value="0.07" />
+  <xacro:property name="hip_hind_offset_x" value="-0.07" />
+  <xacro:property name="hip_offset_y" value="0.055" />
   <xacro:property name="hip_offset_z" value="0.005" />
-  <!-- Head offsets -->
-  <xacro:property name="head_offset_x" value="0.11" />
+  <!-- Head dimensions -->
+  <xacro:property name="head_length" value="0.08" />
+  <xacro:property name="head_width" value="0.065" />
+  <xacro:property name="head_height" value="0.055" />
+  <xacro:property name="head_mass" value="0.15" />
+  <xacro:property name="head_offset_x" value="0.09" />
   <xacro:property name="head_offset_y" value="0.00" />
-  <xacro:property name="head_offset_z" value="0.025" />
-  <!-- Tail offset -->
-  <xacro:property name="tail_offset_x" value="-0.11" />
+  <xacro:property name="head_offset_z" value="0.02" />
+  <!-- Camera dimensions (mounted above head) -->
+  <xacro:property name="camera_length" value="0.025" />
+  <xacro:property name="camera_width" value="0.035" />
+  <xacro:property name="camera_height" value="0.020" />
+  <xacro:property name="camera_mass" value="0.015" />
+  <!-- Tail -->
+  <xacro:property name="tail_offset_x" value="-0.09" />
   <xacro:property name="tail_offset_y" value="0.00" />
-  <xacro:property name="tail_offset_z" value="0.01" />
-  <!-- Component dimensions -->
-  <xacro:property name="rpi_length" value="0.085" />
-  <xacro:property name="rpi_width" value="0.056" />
-  <xacro:property name="rpi_height" value="0.012" />
-  <xacro:property name="hat_length" value="0.085" />
-  <xacro:property name="hat_width" value="0.056" />
+  <xacro:property name="tail_offset_z" value="0.008" />
+  <xacro:property name="tail_length" value="0.08" />
+  <xacro:property name="tail_mass" value="0.015" />
+  <!-- Electronics -->
+  <xacro:property name="rpi_length" value="0.075" />
+  <xacro:property name="rpi_width" value="0.050" />
+  <xacro:property name="rpi_height" value="0.010" />
+  <xacro:property name="rpi_mass" value="0.045" />
+  <xacro:property name="hat_length" value="0.075" />
+  <xacro:property name="hat_width" value="0.050" />
   <xacro:property name="hat_height" value="0.008" />
+  <xacro:property name="hat_mass" value="0.022" />
   <!-- Colors -->
-  <xacro:property name="body_color" value="0.35 0.35 0.35 1.0" />
-  <xacro:property name="leg_color" value="0.25 0.25 0.25 1.0" />
-  <xacro:property name="head_color" value="0.4 0.4 0.4 1.0" />
-  <xacro:property name="snout_color" value="0.3 0.3 0.3 1.0" />
-  <xacro:property name="rpi_color" value="0.0 0.6 0.0 1.0" />
-  <xacro:property name="hat_color" value="0.0 0.0 0.8 1.0" />
-  <xacro:property name="tail_color" value="0.25 0.25 0.25 1.0" />
+  <xacro:property name="body_color" value="0.30 0.30 0.35 1.0" />
+  <xacro:property name="leg_color" value="0.25 0.25 0.28 1.0" />
+  <xacro:property name="head_color" value="0.32 0.32 0.38 1.0" />
+  <xacro:property name="camera_color" value="0.1 0.1 0.1 1.0" />
+  <xacro:property name="rpi_color" value="0.0 0.5 0.0 1.0" />
+  <xacro:property name="hat_color" value="0.0 0.0 0.7 1.0" />
+  <xacro:property name="tail_color" value="0.28 0.28 0.32 1.0" />
+  <xacro:property name="eye_color" value="1.0 1.0 1.0 1.0" />
   <!-- Materials -->
   <material name="body_material"><color rgba="${body_color}" /></material>
   <material name="leg_material"><color rgba="${leg_color}" /></material>
   <material name="head_material"><color rgba="${head_color}" /></material>
-  <material name="snout_material"><color rgba="${snout_color}" /></material>
+  <material name="camera_material"><color rgba="${camera_color}" /></material>
   <material name="rpi_material"><color rgba="${rpi_color}" /></material>
   <material name="hat_material"><color rgba="${hat_color}" /></material>
   <material name="tail_material"><color rgba="${tail_color}" /></material>
-  <material name="eye_material"><color rgba="1.0 1.0 1.0 1.0" /></material>
-  <material name="pupil_material"><color rgba="0.0 0.0 0.0 1.0" /></material>
+  <material name="eye_material"><color rgba="${eye_color}" /></material>
+  <material name="lens_material"><color rgba="0.2 0.5 0.8 1.0" /></material>
+  <!-- ==================== Gazebo Extensions ==================== -->
+  <gazebo>
+    <plugin name="gazebo_ros_control" filename="libgazebo_ros_control.so">
+      <robotNamespace>/pidog</robotNamespace>
+      <controlPeriod>0.01</controlPeriod>
+    </plugin>
+    <static>false</static>
+  </gazebo>
   <!-- ==================== Base Link (Body) ==================== -->
   <link name="base_link">
     <visual>
-      <geometry>
-        <box size="${body_length} ${body_width} ${body_height}" />
-      </geometry>
+      <geometry><box size="${body_length} ${body_width} ${body_height}" /></geometry>
       <origin xyz="0 0 0" />
       <material name="body_material" />
     </visual>
     <collision>
-      <geometry>
-        <box size="${body_length} ${body_width} ${body_height}" />
-      </geometry>
+      <geometry><box size="${body_length} ${body_width} ${body_height}" /></geometry>
+      <origin xyz="0 0 0" />
     </collision>
     <inertial>
       <mass value="${body_mass}" />
       <origin xyz="0 0 0" />
-      <inertia ixx="0.012" ixy="0" ixz="0" iyy="0.012" iyz="0" izz="0.008" />
-    </inertial>
-  </link>
-  <!-- ==================== Raspberry Pi 5 (on top of body) ==================== -->
+      <inertia ixx="0.008" ixy="0" ixz="0" iyy="0.008" iyz="0" izz="0.005" />
+    </inertial>
+  </link>
+  <gazebo reference="base_link">
+    <material>Gazebo/DarkGrey</material>
+    <mu1>0.4</mu1>
+    <mu2>0.4</mu2>
+  </gazebo>
+  <!-- ==================== Raspberry Pi (on top of body) ==================== -->
   <joint name="rpi_joint" type="fixed">
     <origin xyz="0 0 ${body_height/2 + rpi_height/2}" rpy="0 0 0" />
@@ -84,17 +102,19 @@
   <link name="rpi_link">
     <visual>
-      <geometry>
-        <box size="${rpi_length} ${rpi_width} ${rpi_height}" />
-      </geometry>
+      <geometry><box size="${rpi_length} ${rpi_width} ${rpi_height}" /></geometry>
       <origin xyz="0 0 0" />
       <material name="rpi_material" />
     </visual>
-    <inertial>
-      <mass value="0.05" />
-      <origin xyz="0 0 0" />
-      <inertia ixx="0.0001" ixy="0" ixz="0" iyy="0.0001" iyz="0" izz="0.0001" />
-    </inertial>
-  </link>
-  <!-- ==================== Robot HAT Board (above Raspberry Pi) ==================== -->
+    <collision>
+      <geometry><box size="${rpi_length} ${rpi_width} ${rpi_height}" /></geometry>
+      <origin xyz="0 0 0" />
+    </collision>
+    <inertial>
+      <mass value="${rpi_mass}" />
+      <origin xyz="0 0 0" />
+      <inertia ixx="0.00004" ixy="0" ixz="0" iyy="0.00004" iyz="0" izz="0.00004" />
+    </inertial>
+  </link>
+  <!-- ==================== Robot HAT (above Pi) ==================== -->
   <joint name="hat_joint" type="fixed">
     <origin xyz="0 0 ${body_height/2 + rpi_height + hat_height/2}" rpy="0 0 0" />
@@ -104,51 +124,36 @@
   <link name="hat_link">
     <visual>
-      <geometry>
-        <box size="${hat_length} ${hat_width} ${hat_height}" />
-      </geometry>
+      <geometry><box size="${hat_length} ${hat_width} ${hat_height}" /></geometry>
       <origin xyz="0 0 0" />
       <material name="hat_material" />
     </visual>
-    <inertial>
-      <mass value="0.03" />
-      <origin xyz="0 0 0" />
-      <inertia ixx="0.00005" ixy="0" ixz="0" iyy="0.00005" iyz="0" izz="0.00005" />
+    <collision>
+      <geometry><box size="${hat_length} ${hat_width} ${hat_height}" /></geometry>
+      <origin xyz="0 0 0" />
+    </collision>
+    <inertial>
+      <mass value="${hat_mass}" />
+      <origin xyz="0 0 0" />
+      <inertia ixx="0.000025" ixy="0" ixz="0" iyy="0.000025" iyz="0" izz="0.000025" />
     </inertial>
   </link>
   <!-- ==================== Head Assembly ==================== -->
-  <!-- Head roll joint -->
-  <joint name="head_roll_joint" type="revolute">
+  <!-- Head yaw (left/right) -->
+  <joint name="head_yaw_joint" type="revolute">
     <origin xyz="${head_offset_x} ${head_offset_y} ${head_offset_z}" rpy="0 0 0" />
     <parent link="base_link" />
-    <child link="head_yaw_link" />
-    <axis xyz="1 0 0" />
-    <limit lower="-0.5" upper="0.5" effort="1.5" velocity="2.0" />
-  </joint>
-  <link name="head_yaw_link">
-    <visual>
-      <geometry><cylinder radius="0.015" length="0.025" /></geometry>
-      <origin xyz="0 0 0" rpy="1.57 0 0" />
-      <material name="body_material" />
-    </visual>
-    <inertial>
-      <mass value="0.02" />
-      <inertia ixx="0.00005" ixy="0" ixz="0" iyy="0.00005" iyz="0" izz="0.00005" />
-    </inertial>
-  </link>
-  <!-- Head yaw joint -->
-  <joint name="head_yaw_joint" type="revolute">
-    <origin xyz="0 0 0" rpy="0 0 0" />
-    <parent link="head_yaw_link" />
     <child link="head_pitch_link" />
     <axis xyz="0 0 1" />
-    <limit lower="-1.4" upper="1.4" effort="1.5" velocity="2.0" />
+    <limit lower="-1.2" upper="1.2" effort="1.5" velocity="2.5" />
+    <dynamics damping="0.08" friction="0.04" />
   </joint>
   <link name="head_pitch_link">
     <inertial>
-      <mass value="0.015" />
-      <inertia ixx="0.00003" ixy="0" ixz="0" iyy="0.00003" iyz="0" izz="0.00003" />
-    </inertial>
-  </link>
-  <!-- Head pitch joint -->
+      <mass value="0.01" />
+      <origin xyz="0 0 0" />
+      <inertia ixx="0.00001" ixy="0" ixz="0" iyy="0.00001" iyz="0" izz="0.00001" />
+    </inertial>
+  </link>
+  <!-- Head pitch (up/down) -->
   <joint name="head_pitch_joint" type="revolute">
     <origin xyz="0 0 0" rpy="0 0 0" />
@@ -156,5 +161,6 @@
     <child link="head_link" />
     <axis xyz="0 1 0" />
-    <limit lower="-0.7" upper="0.7" effort="1.5" velocity="2.0" />
+    <limit lower="-0.6" upper="0.8" effort="1.5" velocity="2.5" />
+    <dynamics damping="0.08" friction="0.04" />
   </joint>
   <!-- Main head -->
@@ -165,62 +171,76 @@
       <material name="head_material" />
     </visual>
-    <!-- Snout -->
-    <visual name="snout">
-      <geometry><box size="${snout_length} ${head_width*0.6} ${head_height*0.5}" /></geometry>
-      <origin xyz="${head_length/2 + snout_length/2} 0 -${head_height/6}" />
-      <material name="snout_material" />
-    </visual>
     <!-- Eyes -->
     <visual name="left_eye">
-      <geometry><sphere radius="0.007" /></geometry>
-      <origin xyz="${head_length/2 - 0.005} ${head_width/3.5} ${head_height/4}" />
+      <geometry><sphere radius="0.006" /></geometry>
+      <origin xyz="${head_length/2 - 0.005} ${head_width/3.5} ${head_height/5}" />
       <material name="eye_material" />
     </visual>
-    <visual name="left_pupil">
-      <geometry><sphere radius="0.0035" /></geometry>
-      <origin xyz="${head_length/2 - 0.003} ${head_width/3.5} ${head_height/4}" />
-      <material name="pupil_material" />
-    </visual>
     <visual name="right_eye">
-      <geometry><sphere radius="0.007" /></geometry>
-      <origin xyz="${head_length/2 - 0.005} -${head_width/3.5} ${head_height/4}" />
+      <geometry><sphere radius="0.006" /></geometry>
+      <origin xyz="${head_length/2 - 0.005} -${head_width/3.5} ${head_height/5}" />
       <material name="eye_material" />
     </visual>
-    <visual name="right_pupil">
-      <geometry><sphere radius="0.0035}" /></geometry>
-      <origin xyz="${head_length/2 - 0.003} -${head_width/3.5} ${head_height/4}" />
-      <material name="pupil_material" />
-    </visual>
     <collision>
       <geometry><box size="${head_length} ${head_width} ${head_height}" /></geometry>
+      <origin xyz="0 0 0" />
     </collision>
     <inertial>
       <mass value="${head_mass}" />
       <origin xyz="0 0 0" />
-      <inertia ixx="0.0006" ixy="0" ixz="0" iyy="0.0006" iyz="0" izz="0.0006" />
+      <inertia ixx="0.0005" ixy="0" ixz="0" iyy="0.0005" iyz="0" izz="0.0005" />
+    </inertial>
+  </link>
+  <!-- ==================== Camera (on top of head) ==================== -->
+  <joint name="camera_joint" type="fixed">
+    <origin xyz="${head_length/2 - 0.01} 0 ${head_height/2 + camera_height/2}" rpy="0 0 0" />
+    <parent link="head_link" />
+    <child link="camera_link" />
+  </joint>
+  <link name="camera_link">
+    <visual>
+      <geometry><box size="${camera_length} ${camera_width} ${camera_height}" /></geometry>
+      <origin xyz="0 0 0" />
+      <material name="camera_material" />
+    </visual>
+    <!-- Camera lens -->
+    <visual name="lens">
+      <geometry><sphere radius="0.006" /></geometry>
+      <origin xyz="${camera_length/2} 0 0" />
+      <material name="lens_material" />
+    </visual>
+    <collision>
+      <geometry><box size="${camera_length} ${camera_width} ${camera_height}" /></geometry>
+      <origin xyz="0 0 0" />
+    </collision>
+    <inertial>
+      <mass value="${camera_mass}" />
+      <origin xyz="0 0 0" />
+      <inertia ixx="0.000005" ixy="0" ixz="0" iyy="0.000005" iyz="0" izz="0.000005" />
     </inertial>
   </link>
   <!-- ==================== Tail ==================== -->
-  <joint name="tail_base_joint" type="revolute">
+  <joint name="tail_joint" type="revolute">
     <origin xyz="${tail_offset_x} ${tail_offset_y} ${tail_offset_z}" rpy="0 0 0" />
     <parent link="base_link" />
     <child link="tail_link" />
     <axis xyz="0 0 1" />
-    <limit lower="-1.2" upper="1.2" effort="0.8" velocity="3.0" />
+    <limit lower="-1.0" upper="1.0" effort="0.6" velocity="3.0" />
+    <dynamics damping="0.05" friction="0.03" />
   </joint>
   <link name="tail_link">
     <visual>
-      <geometry><cylinder radius="0.007" length="0.095" /></geometry>
-      <origin xyz="0 0 -0.0475" rpy="0.3 0 0" />
+      <geometry><cylinder radius="0.006" length="${tail_length}" /></geometry>
+      <origin xyz="0 0 -${tail_length/2}" rpy="0.2 0 0" />
       <material name="tail_material" />
     </visual>
     <collision>
-      <geometry><cylinder radius="0.007" length="0.095" /></geometry>
-      <origin xyz="0 0 -0.0475" rpy="0.3 0 0" />
-    </collision>
-    <inertial>
-      <mass value="0.02" />
-      <origin xyz="0 0 -0.0475" />
-      <inertia ixx="0.0001" ixy="0" ixz="0" iyy="0.0001" iyz="0" izz="0.00005" />
+      <geometry><cylinder radius="0.006" length="${tail_length}" /></geometry>
+      <origin xyz="0 0 -${tail_length/2}" rpy="0.2 0 0" />
+    </collision>
+    <inertial>
+      <mass value="${tail_mass}" />
+      <origin xyz="0 0 -${tail_length/2}" />
+      <inertia ixx="0.00003" ixy="0" ixz="0" iyy="0.00003" iyz="0" izz="0.000008" />
     </inertial>
   </link>
@@ -233,5 +253,6 @@
       <child link="${prefix}_upper_leg" />
       <axis xyz="0 1 0" />
-      <limit lower="-1.4" upper="1.4" effort="2.0" velocity="3.0" />
+      <limit lower="-1.2" upper="1.2" effort="2.0" velocity="3.0" />
+      <dynamics damping="0.1" friction="0.05" />
     </joint>
     <link name="${prefix}_upper_leg">
@@ -248,5 +269,5 @@
         <mass value="${leg_mass}" />
         <origin xyz="0 -${upper_leg_length/2} 0" />
-        <inertia ixx="0.001" ixy="0" ixz="0" iyy="0.001" iyz="0" izz="0.0005" />
+        <inertia ixx="0.00008" ixy="0" ixz="0" iyy="0.00035" iyz="0" izz="0.00008" />
       </inertial>
     </link>
@@ -257,5 +278,6 @@
       <child link="${prefix}_lower_leg" />
       <axis xyz="0 1 0" />
-      <limit lower="-1.8" upper="0.2" effort="1.5" velocity="3.0" />
+      <limit lower="-1.6" upper="0.1" effort="1.5" velocity="3.0" />
+      <dynamics damping="0.1" friction="0.05" />
     </joint>
     <link name="${prefix}_lower_leg">
@@ -270,7 +292,7 @@
       </collision>
       <inertial>
-        <mass value="${leg_mass*0.8}" />
+        <mass value="${leg_mass*0.7}" />
         <origin xyz="0 -${lower_leg_length/2} 0" />
-        <inertia ixx="0.0008" ixy="0" ixz="0" iyy="0.0008" iyz="0" izz="0.0004" />
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